Commit message: 2.2.0

File: qb_hand_description/urdf/qbhand.utils.xacro (robot description, xacro)
@@ -20,4 +20,16 @@
       </xacro:if>
     </joint>
+    <transmission name="${namespace}_transmission">
+      <type>transmission_interface/qbMoveTransmission</type>
+      <joint name="${namespace}_${finger}_${phalanx}_${virtual_suffix}joint">
+        <hardwareInterface>hardware_interface/EffortJointInterface</hardwareInterface>
+      </joint>
+      <actuator name="${namespace}_${finger}_${phalanx}_${virtual_suffix}joint">
+        <hardwareInterface>hardware_interface/EffortJointInterface</hardwareInterface>
+      </actuator>
+    </transmission>
+    <gazebo reference="${namespace}_${finger}_${phalanx}_${virtual_suffix}joint">
+      <!-- TODO: add other Gazebo Joint properties (http://sdformat.org/spec?elem=joint) -->
+    </gazebo>
   </xacro:macro>
   <xacro:macro name="build_link" params="name **inertia material:=^|'default' mesh:=^|'' mesh_collision:=^|''">
@@ -38,11 +50,33 @@
       </xacro:if>
     </link>
-  </xacro:macro>
-  <xacro:macro name="build_virtual_link" params="name negligible_mass:=^|.01">
+    <gazebo reference="${name}_link">
+      <self_collide>1</self_collide>
+      <!-- TODO: add other Gazebo Link properties (http://sdformat.org/spec?elem=link) -->
+      <!--      <collision>-->
+      <!--        <surface>-->
+      <!--          <contact>-->
+      <!--            <ode>-->
+      <!--              <kp>1.0</kp>-->
+      <!--              <kd>0.01</kd>-->
+      <!--              <max_vel>0.0</max_vel>-->
+      <!--              <min_depth>0.001</min_depth>-->
+      <!--            </ode>-->
+      <!--          </contact>-->
+      <!--          <friction>-->
+      <!--            <ode>-->
+      <!--              <mu>0.9</mu>-->
+      <!--              <mu2>0.9</mu2>-->
+      <!--            </ode>-->
+      <!--          </friction>-->
+      <!--        </surface>-->
+      <!--      </collision>-->
+    </gazebo>
+  </xacro:macro>
+  <xacro:macro name="build_virtual_link" params="name">
     <link name="${name}_virtual_link">
       <inertial>
         <origin xyz="0 0 0" rpy="0 0 0"/>
-        <mass value="${negligible_mass}"/>
-        <inertia ixx="${negligible_mass * 1e-6}" ixy="0.0" ixz="0.0" iyy="${negligible_mass * 1e-6}" iyz="0.0" izz="${negligible_mass * 1e-6}"/>
+        <mass value="1e-4"/>
+        <inertia ixx="1e-9" ixy="0.0" ixz="0.0" iyy="1e-9" iyz="0.0" izz="1e-9"/>
       </inertial>
     </link>
@@ -104,5 +138,6 @@
       <inertial_group>
         <mass value="${yaml_file[configuration][finger][phalanx]['inertial']['mass']}"/>
-        <origin xyz="${yaml_file[configuration][finger][phalanx]['inertial']['origin']}"/>
+        <origin xyz="${yaml_file[configuration][finger][phalanx]['inertial']['origin']['position']}"
+                rpy="${yaml_file[configuration][finger][phalanx]['inertial']['origin']['orientation']}"/>
         <inertia ixx="${yaml_file[configuration][finger][phalanx]['inertial']['inertia']['ixx']}"
                  ixy="${yaml_file[configuration][finger][phalanx]['inertial']['inertia']['ixy']}"
@@ -146,5 +181,6 @@
       <inertial_group>
         <mass value="${yaml_file[configuration][name]['inertial']['mass']}"/>
-        <origin xyz="${yaml_file[configuration][name]['inertial']['origin']}"/>
+        <origin xyz="${yaml_file[configuration][name]['inertial']['origin']['position']}"
+                rpy="${yaml_file[configuration][name]['inertial']['origin']['orientation']}"/>
         <inertia ixx="${yaml_file[configuration][name]['inertial']['inertia']['ixx']}"
                  ixy="${yaml_file[configuration][name]['inertial']['inertia']['ixy']}"
@@ -156,23 +192,32 @@
     </xacro:build_fixed_structure>
   </xacro:macro>
-  <xacro:macro name="build_synergy_mechanism" params="namespace:=^ parent:=^ axis *dynamics *limits">
-    <joint name="${namespace}_synergy_joint" type="revolute">
+  <xacro:macro name="build_synergy_mechanism" params="namespace:=^ synergy_type:=^ parent:=^ axis *dynamics *limits">
+    <joint name="${namespace}_${synergy_type}_joint" type="revolute">
       <origin xyz="0 0 0" rpy="0 0 0"/>
       <parent link="${parent}_link"/>
-      <child link="${namespace}_tendon_virtual_link"/>
+      <child link="${namespace}_${synergy_type}_tendon_virtual_link"/>
       <axis xyz="${axis}"/>
       <xacro:insert_block name="dynamics"/>
       <xacro:insert_block name="limits"/>
     </joint>
-    <xacro:build_virtual_link name="${namespace}_tendon"/>
-  </xacro:macro>
-  <xacro:macro name="build_synergy_mechanism_from_yaml" params="namespace:=^ parent">
-    <xacro:build_synergy_mechanism axis="${yaml_file[configuration]['synergy']['axis']}">
-      <dynamics damping="${yaml_file[configuration]['synergy']['dynamics']['damping']}"
-                friction="${yaml_file[configuration]['synergy']['dynamics']['friction']}"/>
-      <limit lower="${yaml_file[configuration]['synergy']['limits']['lower']}"
-             upper="${yaml_file[configuration]['synergy']['limits']['upper']}"
-             effort="${yaml_file[configuration]['synergy']['limits']['effort']}"
-             velocity="${yaml_file[configuration]['synergy']['limits']['velocity']}"/>
+    <transmission name="${namespace}_${synergy_type}_transmission">
+      <type>transmission_interface/qbMoveTransmission</type>
+      <joint name="${namespace}_${synergy_type}_joint">
+        <hardwareInterface>hardware_interface/EffortJointInterface</hardwareInterface>
+      </joint>
+      <actuator name="${namespace}_${synergy_type}_joint">
+        <hardwareInterface>hardware_interface/EffortJointInterface</hardwareInterface>
+      </actuator>
+    </transmission>
+    <xacro:build_virtual_link name="${namespace}_${synergy_type}_tendon"/>
+  </xacro:macro>
+  <xacro:macro name="build_synergy_mechanism_from_yaml" params="namespace:=^ synergy_type parent">
+    <xacro:build_synergy_mechanism axis="${yaml_file[configuration][synergy_type]['axis']}">
+      <dynamics damping="${yaml_file[configuration][synergy_type]['dynamics']['damping']}"
+                friction="${yaml_file[configuration][synergy_type]['dynamics']['friction']}"/>
+      <limit lower="${yaml_file[configuration][synergy_type]['limits']['lower']}"
+             upper="${yaml_file[configuration][synergy_type]['limits']['upper']}"
+             effort="${yaml_file[configuration][synergy_type]['limits']['effort']}"
+             velocity="${yaml_file[configuration][synergy_type]['limits']['velocity']}"/>
     </xacro:build_synergy_mechanism>
   </xacro:macro>
@@ -186,5 +231,5 @@
     </xacro:build_displaced_fixed_structure_from_yaml>
     <xacro:build_fixed_structure_from_yaml name="palm" parent="${namespace}_base"/>
-    <xacro:build_synergy_mechanism_from_yaml parent="${namespace}_palm"/>
+    <xacro:build_synergy_mechanism_from_yaml synergy_type="synergy" parent="${namespace}_palm"/>
     <xacro:build_two_phalanx_finger_from_yaml finger="thumb" parent="${namespace}_palm"/>
     <xacro:build_three_phalanx_finger_from_yaml finger="index" parent="${namespace}_palm"/>
@@ -193,3 +238,11 @@
     <xacro:build_three_phalanx_finger_from_yaml finger="little" parent="${namespace}_palm"/>
   </xacro:macro>
+  <xacro:macro name="build_hand_2m_from_yaml" params="filename:='default' configuration:='qbhand_right' namespace parent *origin">
+    <xacro:property name="yaml_filename" value="$(find qb_hand_description)/config/${filename}.yaml"/>
+    <xacro:property name="yaml_file" value="${load_yaml(yaml_filename)}"/>
+    <xacro:build_hand_from_yaml filename="${filename}" configuration="${configuration}" namespace="${namespace}" parent="${parent}">
+      <xacro:insert_block name="origin"/>
+    </xacro:build_hand_from_yaml>
+    <xacro:build_synergy_mechanism_from_yaml synergy_type="manipulation" parent="${namespace}_palm"/>
+  </xacro:macro>
 </robot>

File: qb_hand_description/urdf/qbhand2m.urdf.xacro (robot description, xacro)
@@ -1,10 +1,10 @@
 <?xml version="1.0"?>
-<robot name="qbhand" xmlns:xacro="http://www.ros.org/wiki/xacro">
+<robot name="qbhand2m" xmlns:xacro="http://www.ros.org/wiki/xacro">
   <xacro:include filename="$(find qb_hand_description)/urdf/qbhand.utils.xacro"/>
-	<xacro:arg name="namespace" default="qbhand"/>
+	<xacro:arg name="namespace" default="qbhand2m"/>
 	<link name="root_link"/>
-	<xacro:build_hand_from_yaml configuration="qbhand_right" namespace="$(arg namespace)" parent="root">
+	<xacro:build_hand_2m_from_yaml configuration="qbhand_right" namespace="$(arg namespace)" parent="root">
 		<origin xyz="0 0 0" rpy="0 0 0"/>
-	</xacro:build_hand_from_yaml>
+	</xacro:build_hand_2m_from_yaml>
 	<gazebo>
 		<plugin name="qb_hand_gazebo_plugin" filename="libqb_hand_gazebo_plugin.so"/>

Commit message: 2.3.0

File: qb_hand_description/urdf/qbhand.utils.xacro (robot description, xacro)
@@ -160,8 +160,8 @@
     <xacro:build_phalanx_from_yaml phalanx="distal" parent="${namespace}_${finger}_middle"/>
   </xacro:macro>
-  <xacro:macro name="build_fixed_structure" params="name:=^ *origin parent:=^ *inertia material:=^ mesh:=^ mesh_collision:=^">
+  <xacro:macro name="build_fixed_structure" params="name:=^ *origin parent:=^ parent_link_suffix:=^|'_link' *inertia material:=^ mesh:=^ mesh_collision:=^">
     <joint name="${name}_fixed_joint" type="fixed">
       <xacro:insert_block name="origin"/>
-      <parent link="${parent}_link"/>
+      <parent link="${parent}${parent_link_suffix}"/>
       <child link="${name}_link"/>
     </joint>
@@ -170,5 +170,5 @@
     </xacro:build_link>
   </xacro:macro>
-  <xacro:macro name="build_fixed_structure_from_yaml" params="yaml_file:=^ configuration:=^ name namespace:=^ parent">
+  <xacro:macro name="build_fixed_structure_from_yaml" params="yaml_file:=^ configuration:=^ name namespace:=^ parent parent_link_suffix:=^|'_link'">
     <xacro:build_displaced_fixed_structure_from_yaml name="${name}" parent="${parent}">
       <origin xyz="${yaml_file[configuration][name]['position']}"
@@ -176,5 +176,5 @@
     </xacro:build_displaced_fixed_structure_from_yaml>
   </xacro:macro>
-  <xacro:macro name="build_displaced_fixed_structure_from_yaml" params="yaml_file:=^ configuration:=^ name namespace:=^ parent *origin">
+  <xacro:macro name="build_displaced_fixed_structure_from_yaml" params="yaml_file:=^ configuration:=^ name namespace:=^ parent parent_link_suffix:=^|'_link' *origin">
     <xacro:build_fixed_structure name="${namespace}_${name}" material="${name}" mesh="${yaml_file[configuration][name]['mesh']}" mesh_collision="${yaml_file[configuration][name]['mesh_collision']}">
       <xacro:insert_block name="origin"/>
@@ -222,5 +222,5 @@
     </xacro:build_synergy_mechanism>
   </xacro:macro>
-  <xacro:macro name="build_hand_from_yaml" params="filename:='default' configuration:='qbhand_right' namespace parent *origin">
+  <xacro:macro name="build_hand_from_yaml" params="filename:='default' configuration:='qbhand_right' namespace parent parent_link_suffix:=^|'_link' *origin">
     <xacro:property name="use_mimic" value="true"/>
     <xacro:property name="mimic_joint" value="${namespace}_synergy"/>
@@ -230,5 +230,10 @@
       <xacro:insert_block name="origin"/>
     </xacro:build_displaced_fixed_structure_from_yaml>
-    <xacro:build_fixed_structure_from_yaml name="palm" parent="${namespace}_base"/>
+    <xacro:if value="${parent_link_suffix != '_link'}">
+      <xacro:build_fixed_structure_from_yaml name="palm" parent="${namespace}_base_link"/>
+    </xacro:if>
+    <xacro:if value="${parent_link_suffix == '_link'}">
+      <xacro:build_fixed_structure_from_yaml name="palm" parent="${namespace}_base"/>
+    </xacro:if>
     <xacro:build_synergy_mechanism_from_yaml synergy_type="synergy" parent="${namespace}_palm"/>
     <xacro:build_two_phalanx_finger_from_yaml finger="thumb" parent="${namespace}_palm"/>
@@ -238,5 +243,5 @@
     <xacro:build_three_phalanx_finger_from_yaml finger="little" parent="${namespace}_palm"/>
   </xacro:macro>
-  <xacro:macro name="build_hand_2m_from_yaml" params="filename:='default' configuration:='qbhand_right' namespace parent *origin">
+  <xacro:macro name="build_hand_2m_from_yaml" params="filename:='default' configuration:='qbhand_right' namespace parent parent_link_suffix:=^|'_link' *origin">
     <xacro:property name="yaml_filename" value="$(find qb_hand_description)/config/${filename}.yaml"/>
     <xacro:property name="yaml_file" value="${load_yaml(yaml_filename)}"/>

Commit message: 3.0.0

File: qb_hand_description/urdf/qbhand.utils.xacro (robot description, xacro)
@@ -243,4 +243,28 @@
     <xacro:build_three_phalanx_finger_from_yaml finger="little" parent="${namespace}_palm"/>
   </xacro:macro>
+  <xacro:macro name="build_rotated_hand_from_yaml" params="filename:='default' configuration:='qbhand_right' namespace parent parent_link_suffix:=^|'_link' *origin">
+    <xacro:property name="use_mimic" value="true"/>
+    <xacro:property name="mimic_joint" value="${namespace}_synergy"/>
+    <xacro:property name="yaml_filename" value="$(find qb_hand_description)/config/${filename}.yaml"/>
+    <xacro:property name="yaml_file" value="${load_yaml(yaml_filename)}"/>
+    <xacro:build_displaced_fixed_structure_from_yaml name="base" parent="${parent}">
+      <xacro:insert_block name="origin"/>
+    </xacro:build_displaced_fixed_structure_from_yaml>
+    <xacro:build_displaced_fixed_structure_from_yaml name="90_deg_flange_base" parent="${namespace}_base_link">
+      <origin xyz="0 0 0" rpy="-1.57 0 0"/>
+    </xacro:build_displaced_fixed_structure_from_yaml>
+    <xacro:if value="${parent_link_suffix != '_link'}">
+      <xacro:build_fixed_structure_from_yaml name="palm" parent="${namespace}_base_link"/>
+    </xacro:if>
+    <xacro:if value="${parent_link_suffix == '_link'}">
+      <xacro:build_fixed_structure_from_yaml name="palm" parent="${namespace}_base"/>
+    </xacro:if>
+    <xacro:build_synergy_mechanism_from_yaml synergy_type="synergy" parent="${namespace}_palm"/>
+    <xacro:build_two_phalanx_finger_from_yaml finger="thumb" parent="${namespace}_palm"/>
+    <xacro:build_three_phalanx_finger_from_yaml finger="index" parent="${namespace}_palm"/>
+    <xacro:build_three_phalanx_finger_from_yaml finger="middle" parent="${namespace}_palm"/>
+    <xacro:build_three_phalanx_finger_from_yaml finger="ring" parent="${namespace}_palm"/>
+    <xacro:build_three_phalanx_finger_from_yaml finger="little" parent="${namespace}_palm"/>
+  </xacro:macro>
   <xacro:macro name="build_hand_2m_from_yaml" params="filename:='default' configuration:='qbhand_right' namespace parent parent_link_suffix:=^|'_link' *origin">
     <xacro:property name="yaml_filename" value="$(find qb_hand_description)/config/${filename}.yaml"/>
@@ -250,4 +274,16 @@
     </xacro:build_hand_from_yaml>
     <xacro:build_synergy_mechanism_from_yaml synergy_type="manipulation" parent="${namespace}_palm"/>
+    <xacro:build_synergy_mechanism_from_yaml synergy_type="motor_1" parent="${namespace}_palm"/>
+    <xacro:build_synergy_mechanism_from_yaml synergy_type="motor_2" parent="${namespace}_palm"/>
+  </xacro:macro>
+  <xacro:macro name="build_hand_2m_from_yaml_with_90_deg_flange" params="filename:='default' configuration:='qbhand_right' namespace parent parent_link_suffix:=^|'_link' *origin">
+    <xacro:property name="yaml_filename" value="$(find qb_hand_description)/config/${filename}.yaml"/>
+    <xacro:property name="yaml_file" value="${load_yaml(yaml_filename)}"/>
+    <xacro:build_rotated_hand_from_yaml filename="${filename}" configuration="${configuration}" namespace="${namespace}" parent="${parent}">
+      <xacro:insert_block name="origin"/>
+    </xacro:build_rotated_hand_from_yaml>
+    <xacro:build_synergy_mechanism_from_yaml synergy_type="manipulation" parent="${namespace}_palm"/>
+    <xacro:build_synergy_mechanism_from_yaml synergy_type="motor_1" parent="${namespace}_palm"/>
+    <xacro:build_synergy_mechanism_from_yaml synergy_type="motor_2" parent="${namespace}_palm"/>
   </xacro:macro>
 </robot>

Commit message: 3.0.2

File: qb_hand_description/urdf/qbhand.utils.xacro (robot description, xacro)
@@ -242,4 +242,10 @@
     <xacro:build_three_phalanx_finger_from_yaml finger="ring" parent="${namespace}_palm"/>
     <xacro:build_three_phalanx_finger_from_yaml finger="little" parent="${namespace}_palm"/>
+    <joint name="${namespace}_end_effector_fixed_joint" type="fixed">
+      <origin xyz="-0.03 0.060 0.142" rpy="-1.57 0 0"/>
+      <parent link="${namespace}_base_link"/>
+      <child link="${namespace}_end_effector_link"/>
+    </joint>
+    <link name="${namespace}_end_effector_link"/>
   </xacro:macro>
   <xacro:macro name="build_rotated_hand_from_yaml" params="filename:='default' configuration:='qbhand_right' namespace parent parent_link_suffix:=^|'_link' *origin">
@@ -277,4 +283,11 @@
     <xacro:build_synergy_mechanism_from_yaml synergy_type="motor_2" parent="${namespace}_palm"/>
   </xacro:macro>
+  <xacro:macro name="build_hand_from_yaml_with_90_deg_flange" params="filename:='default' configuration:='qbhand_right' namespace parent parent_link_suffix:=^|'_link' *origin">
+    <xacro:property name="yaml_filename" value="$(find qb_hand_description)/config/${filename}.yaml"/>
+    <xacro:property name="yaml_file" value="${load_yaml(yaml_filename)}"/>
+    <xacro:build_rotated_hand_from_yaml filename="${filename}" configuration="${configuration}" namespace="${namespace}" parent="${parent}">
+      <xacro:insert_block name="origin"/>
+    </xacro:build_rotated_hand_from_yaml>
+  </xacro:macro>
   <xacro:macro name="build_hand_2m_from_yaml_with_90_deg_flange" params="filename:='default' configuration:='qbhand_right' namespace parent parent_link_suffix:=^|'_link' *origin">
     <xacro:property name="yaml_filename" value="$(find qb_hand_description)/config/${filename}.yaml"/>
